Commit message: 优化

File: urdf/chassis.urdf (robot description, URDF)
Before this commit: robot smartcar, 5 links, 4 joints
Joints:
- joint back_left_joint: origin xyz=-0.4 0.35 -0.03 rpy=1.57079 0 0 -> xyz=-0.4 0.35 -0.03 rpy=-1.57079 0 0
- joint back_right_joint: origin xyz=-0.4 -0.35 -0.03 rpy=1.57079 0 0 -> xyz=-0.4 -0.35 -0.03 rpy=-1.57079 0 0
- joint front_left_joint: origin xyz=0.4 0.35 -0.03 rpy=1.57079 0 0 -> xyz=0.4 0.35 -0.03 rpy=-1.57079 0 0
- joint front_right_joint: origin xyz=0.4 -0.35 -0.03 rpy=1.57079 0 0 -> xyz=0.4 -0.35 -0.03 rpy=-1.57079 0 0

Commit message: 备份

File: urdf/chassis.urdf (robot description, URDF)
Before this commit: robot chassis, 5 links, 4 joints
Links:
- link base_link: mass 19.31 -> 46.034
- link left_back_wheel: mass 0.59 -> 2
- link left_front_wheel: mass 0.59 -> 2
- link right_back_wheel: mass 0.59 -> 2
- link right_front_wheel: mass 0.59 -> 2

Commit message: fix

File: urdf/chassis.urdf (robot description, URDF)
Before this commit: robot chassis, 5 links, 4 joints
Links:
- link base_link: geometry collision box size=0.954 0.48 0.181; visual box size=0.954 0.48 0.181
Joints:
- joint back_left_joint: origin xyz=-0.4 0.35 -0.03 rpy=-1.57079 0 0 -> xyz=-0.35 0.2965 -0.059 rpy=-1.57079 0 0
- joint back_right_joint: origin xyz=-0.4 -0.35 -0.03 rpy=-1.57079 0 0 -> xyz=-0.35 -0.2965 -0.059 rpy=-1.57079 0 0
- joint front_left_joint: origin xyz=0.4 0.35 -0.03 rpy=-1.57079 0 0 -> xyz=0.35 0.2965 -0.059 rpy=-1.57079 0 0
- joint front_right_joint: origin xyz=0.4 -0.35 -0.03 rpy=-1.57079 0 0 -> xyz=0.35 -0.2965 -0.059 rpy=-1.57079 0 0
